File: _autosave-lampDriver.kicad_sch (KiCad schematic)
At the start: 56 parts, among them IC8 FAN3100TSX, Q4 BC807, T4 NMOS_GDS-KS_SMD, U1 OPA2356AIDGKR, U3 LM2902

Commit message: error correction
Parts:
- U1: footprint Package_SO:VSSOP-8_3x3mm_P0.65mm -> Package_SO:VSSOP-8_3.0x3.0mm_P0.65mm
Changed lines of the file:
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@@
 			)
 		)
-		(property "Footprint" "Package_SO:VSSOP-8_3x3mm_P0.65mm"
+		(property "Footprint" "Package_SO:VSSOP-8_3.0x3.0mm_P0.65mm"
 			(at 250.19 97.79 0)
 			(hide yes)
@@
 			)
 		)
-		(property "Footprint" "Package_SO:VSSOP-8_3x3mm_P0.65mm"
+		(property "Footprint" "Package_SO:VSSOP-8_3.0x3.0mm_P0.65mm"
 			(at 251.46 97.79 0)
 			(hide yes)
@@
 			)
 		)
-		(property "Footprint" "Package_SO:VSSOP-8_3x3mm_P0.65mm"
+		(property "Footprint" "Package_SO:VSSOP-8_3.0x3.0mm_P0.65mm"
 			(at 199.39 100.33 0)
 			(hide yes)
