File: _autosave-offlineConverter.kicad_sch (KiCad schematic)
At the start: 72 parts, among them IC1 NCP12510ASN65T1G, IC2 SFH6156-3, J5 640445-2, Q1 STD3NK80ZT4, Q2 BAT847B, T1 750343466, U2 AZ431LANTR

Commit message: error correction
Parts:
- renumbered T1 to L104
Changed lines of the file:
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@@
 		(dnp no)
 		(fields_autoplaced yes)
-		(property "Reference" "T1"
-			(at 179.07 95.25 0)
+		(property "Reference" "L104"
+			(at 179.07 96.52 0)
 			(effects
 				(font
@@
 		)
 		(property "Value" "750343466"
-			(at 179.07 97.79 0)
+			(at 179.07 99.06 0)
 			(effects
 				(font
@@
 			(project "OSLUV"
 				(path "/c6e900e0-9399-44f0-8089-9dd7b8ffe54c/a8d7965e-5268-4c95-93ca-40f8dbbf325c"
-					(reference "T1")
+					(reference "L104")
 					(unit 1)
 				)
