File: offlineConverter.kicad_sch (KiCad schematic)
At the start: 72 parts, among them IC1 NCP12510ASN65T1G, IC2 SFH6156-3, J5 640445-2, Q1 STD3NK80ZT4, Q2 BAT847B, T1 750343466, U2 AZ431LANTR

Commit message: alpha prototype
Parts:
- C9: value 100pF NP0 0603 -> 100pF NP0 1206
- R26: value 51 0805 -> 51R 0805
- renumbered T1 to L104
Changed lines of the file:
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@@
 		(polyline
 			(pts
-				(xy 21.59 29.21) (xy 21.59 73.66) (xy 52.07 73.66) (xy 52.07 33.655) (xy 52.07 29.21)
+				(xy 165.1 110.49) (xy 165.1 77.47) (xy 24.13 77.47) (xy 24.13 109.22) (xy 36.83 109.22) (xy 36.83 85.09)
+				(xy 87.63 85.09) (xy 87.63 110.49) (xy 92.71 110.49)
 			)
 			(stroke
@@
 		(polyline
 			(pts
-				(xy 165.1 110.49) (xy 165.1 77.47) (xy 24.13 77.47) (xy 24.13 109.22) (xy 36.83 109.22) (xy 36.83 85.09)
-				(xy 87.63 85.09) (xy 87.63 110.49) (xy 92.71 110.49)
+				(xy 21.59 29.21) (xy 21.59 73.66) (xy 52.07 73.66) (xy 52.07 33.655) (xy 52.07 29.21)
 			)
 			(stroke
@@
 			)
 		)
-		(property "Value" "51 0805"
+		(property "Value" "51R 0805"
 			(at 256.54 142.494 90)
 			(effects
@@
 			)
 		)
-		(property "Value" "100pF NP0 0603"
+		(property "Value" "100pF NP0 1206"
 			(at 94.996 81.026 0)
 			(effects
@@
 		(dnp no)
 		(fields_autoplaced yes)
-		(property "Reference" "T1"
-			(at 179.07 95.25 0)
+		(property "Reference" "L104"
+			(at 179.07 96.52 0)
 			(effects
 				(font
@@
 		)
 		(property "Value" "750343466"
-			(at 179.07 97.79 0)
+			(at 179.07 99.06 0)
 			(effects
 				(font
@@
 			(project "OSLUV"
 				(path "/c6e900e0-9399-44f0-8089-9dd7b8ffe54c/a8d7965e-5268-4c95-93ca-40f8dbbf325c"
-					(reference "T1")
+					(reference "L104")
 					(unit 1)
 				)

Commit message: V2 PCB
Parts:
- removed Q2: BAT847B, Package_TO_SOT_SMD:SOT-23, symbol Simulation_SPICE:NPN
- added Q6: BC847, Package_TO_SOT_SMD:SOT-23, symbol Transistor_BJT:BC847
Connections:
- net at C11.1, C12.1, C13.2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: now also Q6.3 (C)
- net at D3.2 (A): now also Q6.2 (E)
- net at D4.1 (K), R12.2: now also Q6.1 (B)
